File: RFamp-PCB/RFamp-PCB.kicad_sch (KiCad schematic)
At the start: 0 parts

Commit message: schematic mostly done
Parts:
- added C1, C7: 1u, symbol Device:C
- added C2, C3: 100p, symbol Device:C
- added C4: 2p4, symbol Device:C
- added C5: 1n, symbol Device:C
- added C6: 220p, symbol Device:C
- added C8: 4u7, symbol Device:C
- added C9: 18p, symbol Device:C
- added D1: D, symbol Device:D
- added J1: 5V_SUPPLY, symbol Connector:Conn_01x02_Pin
- added J2: RF_IN, symbol Connector:Conn_Coaxial_Small
- added J3: P_DET, symbol Connector:Conn_01x02_Pin
- added J4: RF_OUT, symbol Connector:Conn_Coaxial_Small
- added L1: 3n9, symbol Device:L
- added L2: 12n, symbol Device:L
- added L3, L5: 5n6, symbol Device:L
- added L4: 22n, symbol Device:L
- added R1: 1k8, symbol Device:R
- added R2: 2k, symbol Device:R
- added U1: MMZ09332BT1, Package_DFN_QFN:QFN-12-1EP_3x3mm_P0.5mm_EP1.6x1.6mm_ThermalVias, symbol RF_Amplifier:MMZ09332BT1
Connections:
- new net: C9.2, J4.1 (In), L5.2
- new net: C6.2, L4.1, L5.1
- new net: R1.2, U1.1 (VBA1)
- new net: C4.1, L3.1, U1.11 (VCC1)
- new net: R2.2, U1.12 (VBA2)
- new net: L1.2, U1.3 (RF_IN)
- new net: C2.1, J3.2 (Pin_2), U1.6 (PDET)
- new net: C6.1, L2.1, U1.7 (VCC2/RFOUT), U1.8 (VCC2/RFOUT), U1.9 (VCC2/RFOUT)
- new net: J2.1 (In), L1.1
- new net: D1.2 (A), J1.1 (Pin_1)
- new net GND: C1.2, C2.2, C3.2, C4.2, C5.1, C7.2, C8.1, C9.1, J1.2 (Pin_2), J2.2 (Ext), J3.1 (Pin_1), J4.2 (Ext), L4.2, U1.13 (GND)
- new net VCC1: C1.1, C3.1, C5.2, C7.1, C8.2, D1.1 (K), L2.2, L3.2, R1.1, R2.1, U1.2 (VBIAS)
